Commit message: URDF file now loads parameters from yaml config file

File: turtle_brick/urdf/turtle.urdf.xacro (robot description, xacro)
@@ -1,7 +1,18 @@
 <robot name="turtle" xmlns:xacro="http://www.ros.org/wiki/xacro">
+<xacro:property name="yaml_file" value="$(find turtle_brick)/turtle.yaml" />
+<xacro:property name="props" value="${xacro.load_yaml(yaml_file)}"/>
+<xacro:property name="b_dim" value="1"/>
+<xacro:property name="sr" value="0.2"/>
+<xacro:property name="sl" value="0.5"/>
+<xacro:property name="wr" value="${props['wheel_radius']}"/>
+<xacro:property name="wl" value="0.3"/>
+<xacro:property name="pr" value="1"/>
+<xacro:property name="pl" value="0.1"/>
+<xacro:property name="lr" value="0.1"/>
+<xacro:property name="ll" value="${props['platform_height'] - b_dim - sl - 2*wr}"/>
     <link name="base_link">
         <visual>
             <geometry>
-                <box size="1.0 1.0 1.0"/>
+                <box size="${b_dim} ${b_dim} ${b_dim}"/>
             </geometry>
             <material name="green_mat">
@@ -13,5 +24,5 @@
         <visual>
             <geometry>
-                <cylinder radius="0.2" length="0.5" />
+                <cylinder radius="${sr}" length="${sl}" />
             </geometry>
             <material name="blue_mat">
@@ -21,5 +32,5 @@
     </link>
     <joint name="base_to_stem" type="continuous">
-        <origin xyz="0 0 -0.75"/>
+        <origin xyz="0 0 ${-1/2*(b_dim+sl)}"/>
         <axis xyz="0 0 -1"/>
         <parent link="base_link"/>
@@ -30,5 +41,5 @@
             <origin rpy="1.571 0 0"/>
             <geometry>
-                <cylinder radius="0.5" length="0.3"/>
+                <cylinder radius="${wr}" length="${wl}"/>
             </geometry>
             <material name="red_mat">
@@ -37,6 +48,7 @@
         </visual>
     </link>
-    <joint name="stem_to_wheel" type="fixed">
-        <origin xyz="0 0 -0.75"/>
+    <joint name="stem_to_wheel" type="continuous">
+        <origin xyz="0 0 ${-1/2*sl-wr}"/>
+        <axis xyz="0 1 0"/>
         <parent link="stem"/>
         <child link="wheel"/>
@@ -45,5 +57,5 @@
         <visual>
             <geometry>
-                <cylinder radius="0.1" length="1"/>
+                <cylinder radius="${lr}" length="${ll}"/>
             </geometry>
         <material name="black_mat">
@@ -53,5 +65,5 @@
     </link>
     <joint name="base_to_pstem" type="fixed">
-        <origin xyz="0 0 1"/>
+        <origin xyz="0 0 ${1/2*(b_dim+ll)}"/>
         <parent link="base_link"/>
         <child link="platform_stem"/>
@@ -60,14 +72,14 @@
         <visual>
             <geometry>
-                <cylinder radius="1" length="0.1"/>
+                <cylinder radius="${pr}" length="${pl}"/>
             </geometry>
-            <material name="purple_mat">
-            <color rgba="1 0 1 0.5"/>
-            </material>
+        <material name="purple_mat">
+        <color rgba="1 0 1 0.5"/>
+        </material>
         </visual>
     </link>
     <joint name="pstem_to_platform" type="continuous">
-        <origin xyz="0 0 0.55"/>
-        <axis xyz="1 0 0"/>
+        <origin xyz="0 0 ${1/2*(ll+pl)}" rpy="0 0 1.572"/>
+        <axis xyz="0 1 0"/>
         <parent link="platform_stem"/>
         <child link="platform"/>

Commit message: YAML file parameters now compatible with multiple nodes and fully integrated into current code

File: turtle_brick/urdf/turtle.urdf.xacro (robot description, xacro)
@@ -5,10 +5,10 @@
 <xacro:property name="sr" value="0.2"/>
 <xacro:property name="sl" value="0.5"/>
-<xacro:property name="wr" value="${props['wheel_radius']}"/>
+<xacro:property name="wr" value="${props['/**']['ros__parameters']['wheel_radius']}"/>
 <xacro:property name="wl" value="0.3"/>
 <xacro:property name="pr" value="1"/>
 <xacro:property name="pl" value="0.1"/>
 <xacro:property name="lr" value="0.1"/>
-<xacro:property name="ll" value="${props['platform_height'] - b_dim - sl - 2*wr}"/>
+<xacro:property name="ll" value="${props['/**']['ros__parameters']['platform_height'] - b_dim - sl - 2*wr}"/>
     <link name="base_link">
         <visual>
@@ -33,5 +33,5 @@
     <joint name="base_to_stem" type="continuous">
         <origin xyz="0 0 ${-1/2*(b_dim+sl)}"/>
-        <axis xyz="0 0 -1"/>
+        <axis xyz="0 0 -1" rpy="0 ${pi} 0"/>
         <parent link="base_link"/>
         <child link="stem"/>
